File: PCB/LED_Board_Base/LED_Board_Base.kicad_sch (KiCad schematic)
At the start: 45 parts, among them J1 Conn_01x02_Socket, J10 Conn_01x02_Socket, J2 Conn_01x02_Socket, J3 Conn_01x02_Socket, J4 Conn_01x02_Socket, J5 Conn_01x02_Socket, J6 Conn_01x02_Socket, J7 Conn_01x02_Socket, J8 Conn_01x02_Socket, J9 Conn_01x02_Socket, SW1 SW_SPDT, SW10 SW_SPDT, SW11 SW_SPDT, SW12 SW_SPDT, SW13 SW_SPDT, SW2 SW_SPDT, SW3 SW_SPDT, SW4 SW_SPDT, SW5 SW_SPDT, SW6 SW_SPDT, SW7 SW_SPDT, SW8 SW_SPDT, SW9 SW_SPDT, U1 RP2040-ZERO

Commit message: schematic pdf
Parts:
- J4: value Conn_01x02_Socket -> 01x02 Solder Wire
- J5, J6, J7, J8, J9: value Conn_01x02_Socket -> Screw Terminal
Other:
- company: (none) -> UMD DBF 2027
- title: (none) -> LED Tester 9000
- moved on the sheet: J4, J5
Changed lines of the file:
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@@
 	(generator "eeschema")
 	(generator_version "9.0")
-	(paper "A4")
+	(paper "USLetter")
+	(title_block
+		(title "LED Tester 9000")
+		(date "2026-10-13")
+		(rev "1")
+		(company "UMD DBF 2027")
+		(comment 1 "Designed by Shawn Malluwa-Wadu")
+	)
 	(junction
 		(at 213.36 97.79)
@@
 	)
 	(junction
-		(at 255.27 38.1)
+		(at 234.95 60.96)
 		(diameter 0)
 		(color 0 0 0 0)
@@
 	(wire
 		(pts
-			(xy 259.08 24.13) (xy 252.73 24.13)
+			(xy 238.76 46.99) (xy 232.41 46.99)
 		)
 		(stroke
@@
 	(wire
 		(pts
-			(xy 255.27 38.1) (xy 259.08 38.1)
+			(xy 234.95 60.96) (xy 238.76 60.96)
 		)
 		(stroke
@@
 	(wire
 		(pts
-			(xy 252.73 24.13) (xy 252.73 35.56)
+			(xy 232.41 46.99) (xy 232.41 58.42)
 		)
 		(stroke
@@
 	(wire
 		(pts
-			(xy 259.08 35.56) (xy 252.73 35.56)
+			(xy 238.76 58.42) (xy 232.41 58.42)
 		)
 		(stroke
@@
 	(wire
 		(pts
-			(xy 255.27 26.67) (xy 255.27 38.1)
+			(xy 234.95 49.53) (xy 234.95 60.96)
 		)
 		(stroke
@@
 	(wire
 		(pts
-			(xy 259.08 26.67) (xy 255.27 26.67)
+			(xy 238.76 49.53) (xy 234.95 49.53)
 		)
 		(stroke
@@
 			)
 		)
-		(property "Value" "Conn_01x02_Socket"
+		(property "Value" "Screw Terminal"
 			(at 119.38 18.4149 90)
 			(effects
@@
 	(symbol
 		(lib_id "Connector:Conn_01x02_Socket")
-		(at 264.16 24.13 0)
+		(at 243.84 46.99 0)
 		(unit 1)
 		(exclude_from_sim no)
@@
 		(fields_autoplaced yes)
 		(property "Reference" "J4"
-			(at 265.43 24.1299 0)
+			(at 245.11 46.9899 0)
 			(effects
 				(font
@@
 			)
 		)
-		(property "Value" "Conn_01x02_Socket"
-			(at 265.43 26.6699 0)
+		(property "Value" "01x02 Solder Wire"
+			(at 245.11 49.5299 0)
 			(effects
 				(font
@@
 		)
 		(property "Footprint" "Connector_Wire:SolderWire-1sqmm_1x02_P7.8mm_D1.4mm_OD3.9mm_Relief"
-			(at 264.16 24.13 0)
+			(at 243.84 46.99 0)
 			(effects
 				(font
@@
 		)
 		(property "Datasheet" "~"
-			(at 264.16 24.13 0)
+			(at 243.84 46.99 0)
 			(effects
 				(font
@@
 		)
 		(property "Description" "Generic connector, single row, 01x02, script generated"
-			(at 264.16 24.13 0)
+			(at 243.84 46.99 0)
 			(effects
 				(font
@@
 			)
 		)
-		(property "Value" "Conn_01x02_Socket"
+		(property "Value" "Screw Terminal"
 			(at 149.86 74.2949 90)
 			(effects
@@
 	(symbol
 		(lib_id "power:GND")
-		(at 255.27 38.1 0)
+		(at 234.95 60.96 0)
 		(unit 1)
 		(exclude_from_sim no)
@@
 		(fields_autoplaced yes)
 		(property "Reference" "#PWR06"
-			(at 255.27 44.45 0)
+			(at 234.95 67.31 0)
 			(effects
 				(font
@@
 		)
 		(property "Value" "GND"
-			(at 255.27 43.18 0)
+			(at 234.95 66.04 0)
 			(effects
 				(font
@@
 		)
 		(property "Footprint" ""
-			(at 255.27 38.1 0)
+			(at 234.95 60.96 0)
 			(effects
 				(font
@@
 		)
 		(property "Datasheet" ""
-			(at 255.27 38.1 0)
+			(at 234.95 60.96 0)
 			(effects
 				(font
@@
 		)
 		(property "Description" "Power symbol creates a global label with name \"GND\" , ground"
-			(at 255.27 38.1 0)
+			(at 234.95 60.96 0)
 			(effects
 				(font
@@
 			)
 		)
-		(property "Value" "Conn_01x02_Socket"
+		(property "Value" "Screw Terminal"
 			(at 217.17 74.2949 90)
 			(effects
@@
 			)
 		)
-		(property "Value" "Conn_01x02_Socket"
+		(property "Value" "Screw Terminal"
 			(at 85.09 74.2949 90)
 			(effects
@@
 	(symbol
 		(lib_id "Connector:Conn_01x02_Socket")
-		(at 264.16 35.56 0)
+		(at 243.84 58.42 0)
 		(unit 1)
 		(exclude_from_sim no)
@@
 		(fields_autoplaced yes)
 		(property "Reference" "J5"
-			(at 265.43 35.5599 0)
+			(at 245.11 58.4199 0)
 			(effects
 				(font
@@
 			)
 		)
-		(property "Value" "Conn_01x02_Socket"
-			(at 265.43 38.0999 0)
+		(property "Value" "Screw Terminal"
+			(at 245.11 60.9599 0)
 			(effects
 				(font
@@
 		)
 		(property "Footprint" "TerminalBlock:TerminalBlock_MaiXu_MX126-5.0-02P_1x02_P5.00mm"
-			(at 264.16 35.56 0)
+			(at 243.84 58.42 0)
 			(effects
 				(font
@@
 		)
 		(property "Datasheet" "~"
-			(at 264.16 35.56 0)
+			(at 243.84 58.42 0)
 			(effects
 				(font
@@
 		)
 		(property "Description" "Generic connector, single row, 01x02, script generated"
-			(at 264.16 35.56 0)
+			(at 243.84 58.42 0)
 			(effects
 				(font
