File: PCB/LED_Board_Base/LED_Board_Base.kicad_pcb (KiCad board)
At the start: 2 copper layers, 118 x 69 mm, 45 parts, among them J1 Conn_01x02_Socket, J10 Conn_01x02_Socket, J2 Conn_01x02_Socket, J3 Conn_01x02_Socket, J4 Conn_01x02_Socket, J5 Conn_01x02_Socket, J6 Conn_01x02_Socket, J7 Conn_01x02_Socket, J8 Conn_01x02_Socket, J9 Conn_01x02_Socket, SW1 SW_SPDT, SW10 SW_SPDT, SW11 SW_SPDT, SW12 SW_SPDT, SW13 SW_SPDT, SW2 SW_SPDT, SW3 SW_SPDT, SW4 SW_SPDT, SW5 SW_SPDT, SW6 SW_SPDT, SW7 SW_SPDT, SW8 SW_SPDT, SW9 SW_SPDT, U1 RP2040-ZERO

Commit message: finished LED testing PCB
Routing:
- net unconnected-(D9-PAD-Pad3): vias 0 -> 10
- net unconnected-(D8-PAD-Pad3): vias 0 -> 7
- net unconnected-(D7-PAD-Pad3): vias 0 -> 7
- net unconnected-(D6-PAD-Pad3): vias 0 -> 7
- net unconnected-(D5-PAD-Pad3): vias 0 -> 7
- net unconnected-(D4-PAD-Pad3): vias 0 -> 7
- net unconnected-(D3-PAD-Pad3): vias 0 -> 7
- net unconnected-(D2-PAD-Pad3): vias 0 -> 7
- net unconnected-(D18-PAD-Pad3): vias 0 -> 7
- net unconnected-(D17-PAD-Pad3): vias 0 -> 7
- net unconnected-(D16-PAD-Pad3): vias 0 -> 7
- net unconnected-(D15-PAD-Pad3): vias 0 -> 7
- net unconnected-(D14-PAD-Pad3): vias 0 -> 7
- net unconnected-(D13-PAD-Pad3): vias 0 -> 10
- net unconnected-(D12-PAD-Pad3): vias 0 -> 10
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Other:
- outline, holes or cut-outs redrawn
- board text added: "GA CS8PM1.23-LPLR- W3-0-350-R18"
- board text added: "GY CSHPM1.23-KQKS- 36-0-350-R18"
- board text added: "KP CSLNM1.F1-8N7P- A-0-1000-R18"
- board text added: "LE CG Q8WP-7P6Q- 2-0-A40-R18-ZI"
- board text added: "LED TESTER 9000"
- board text added: "POWER"
- board text added: "XPEBRD-L1-0000-00501"

Commit message: via fixes
Routing:
- net unconnected-(D3-PAD-Pad3): track 0.00 -> 42.0 mm, vias 7 -> 9
- net unconnected-(D2-PAD-Pad3): track 0.00 -> 32.3 mm, vias 7 -> 9
- net GND: track 8.83 -> 13.9 mm, vias 0 -> 4
Other:
- board text added: "LED TESTER UMD DBF 2027"
- board text removed: "LED TESTER 9000"
